File: projects_records/White_Noice_Gen/Version1.0/White_noise_generator/White_noise_generator.kicad_sch (KiCad schematic)
At the start: 17 parts, among them J1 Conn_Coaxial, J2 Conn_01x02_Pin, J3 Barrel_Jack, U1 LM2940IMP-9.0_NOPB, U2 LM2940CSX-15_NOPB

Commit message: Jun 30, 2026, 4:39 PM
Parts:
- U2: DESCRIPTION 1A Low Dropout Regulator -> (none)
